File: Hardware/Akkucheck.brd (EAGLE design)
At the start: 21.1 x 17.8 mm, 44 parts, among them IC1 MEGA8-MI, IC2 78L05F

Commit message: updated BOM
Parts:
- C5, C7: value (none) -> 2u2
- moved C5 0.07 mm to (11.8, 15.2)
