File: Hardware/Akkucheck.sch (EAGLE design)
At the start: 44 parts, among them IC1 MEGA8-MI, IC2 78L05F

Commit message: updated BOM
Parts:
- C5, C7: value (none) -> 2u2; MF (none) -> MULTICOMP; MPN (none) -> MC0805B225K250CT; OC_FARNELL (none) -> 2320829
- IC1: MPN ATMEGA88PA-MU -> (none); OC_FARNELL 1715491 -> (none)
- IC2: MF (none) -> STMICROELECTRONICS; MPN (none) -> L78L05ABUTR; OC_FARNELL (none) -> 1467762
- LED1: OC_FARNELL (none) -> unknown
- R1, R11, R12, R5, R7, R9: MF (none) -> TE CONNECTIVITY; MPN (none) -> CRG0402F33K; OC_FARNELL (none) -> 2331513
- R10, R13, R14, R2, R6, R8: MF (none) -> TE CONNECTIVITY; MPN (none) -> CRG0402F8K2; OC_FARNELL (none) -> 2331571
- R15, R17, R18: MF WELWYN -> PANASONIC ELECTRONIC COMPONENTS; MPN ASC0603-470RFT5 -> ERJ2GEJ470X; OC_FARNELL 2078905 -> 2059203
- R16, R20: MF VISHAY DRALORIC -> PANASONIC ELECTRONIC COMPONENTS; MPN CRCW060347K0FKEA -> ERJ2GEJ473X; OC_FARNELL 1469811 -> 2059246
- R19, R21: MF (none) -> PANASONIC ELECTRONIC COMPONENTS; MPN (none) -> ERJ2GEJ102X; OC_FARNELL (none) -> 2059225
- R3: MPN CRCW060310K0FKEA -> CRCW040210K0FKEAHP; OC_FARNELL 1469748 -> 1738864
- R4: MF VISHAY DRALORIC -> PANASONIC ELECTRONIC COMPONENTS; MPN CRCW06032K20FKEA -> ERJ2GEJ222X; OC_FARNELL 1469765 -> 2059231
- T1: MPN BC817 -> BC817,215
